File: Hardware/TuringMachine.brd (EAGLE design)
At the start: 107 x 49.5 mm, 83 parts, among them IC1 TL072P, IC2 4015, IC3 4015, IC5 4016, IC6 TL072P, IC7 TL072P, T1 2N3904, T2 2N3904, T3 2N3904

Commit message: routing
Parts:
- moved D2 76.8 mm to (84.5, 33.0), turned to 90 degrees
- moved R7 67.6 mm to (77.5, 34.3)
- moved R3 67.5 mm to (84.5, 43.2), turned to 90 degrees
- moved C16 62.5 mm to (77.5, 36.8)
- moved R9 57.1 mm to (71.1, 36.8), turned to 90 degrees
- moved C4 31.8 mm to (33.7, 45.7), turned to 90 degrees
- moved IC3 1.27 mm to (91.4, 38.1)
Connections:
- net GND: now also C16.2, R9.2; no longer C16.1, R9.1
- net N$12: now also C16.1, R9.1; no longer C16.2, R9.2
Routing:
- net N$10: track 7.40 -> 6.13 mm
- net B5: track 9.94 -> 8.79 mm

Commit message: routing
Parts:
- moved R12 64.7 mm to (84.5, 23.5), turned to 90 degrees
- moved C7 44.5 mm to (61.0, 21.6), turned to 0 degrees
- moved C8 41.9 mm to (53.3, 21.6), turned to 0 degrees
- moved C14 34.3 mm to (68.6, 34.3)
- moved C13 33.5 mm to (66.0, 34.3)
- moved C15 5.12 mm to (17.8, 33.0)
- moved C2 5.12 mm to (17.1, 38.1)
- moved R10 5.08 mm to (15.9, 35.6)
- moved R14 5.08 mm to (15.9, 40.6)
- turned CLK to 180 degrees
Routing:
- net CLOCKIN: track 0.00 -> 74.7 mm
- net +12V: track 97.7 -> 150.5 mm, vias 0 -> 1
- net N$28: track 0.00 -> 30.0 mm
- net B1: track 10.7 -> 36.4 mm
- net END_OF_LOOP: track 22.0 -> 40.3 mm
- net STEP_16: track 0.00 -> 17.4 mm
- net N$29: track 0.00 -> 8.67 mm
- net N$5: track 0.00 -> 8.19 mm
- net N$15: track 0.00 -> 6.24 mm
- net STEP_12: track 9.40 -> 9.99 mm

Commit message: Prototype 1 complete and sent to OSHPark
Parts:
- moved C7 38.7 mm to (22.2, 22.2)
- moved C8 31.3 mm to (22.2, 24.8)
- moved R30 10.5 mm to (35.6, 11.4)
- moved R29 10.2 mm to (29.2, 15.2)
- moved C18 8.98 mm to (36.8, 16.5), turned to 90 degrees
- moved C5 8.13 mm to (17.1, 18.4), flipped to the top
- moved T1 8.03 mm to (22.9, 16.5)
- moved C10 7.41 mm to (33.0, 16.5), turned to 90 degrees
- moved C6 5.71 mm to (17.1, 28.6), flipped to the top
- moved C11 3.59 mm to (48.3, 7.62), turned to 90 degrees
- moved WRITE 2.54 mm to (39.4, 6.35)
- moved R26 1.27 mm to (68.6, 43.2)
- moved R27 1.27 mm to (66.0, 43.2)
- moved R31 1.27 mm to (45.7, 12.7)
- moved VR2 1.27 mm to (77.5, 26.0)
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Connections:
- net N$22: now also C18.1; no longer C18.2
- net N$9: now also C18.2; no longer C18.1
Routing:
- net GND: track 0.00 -> 376.9 mm, vias 0 -> 1
- net B4: track 0.00 -> 119.0 mm, vias 0 -> 2
- net B1: track 36.4 -> 152.9 mm, vias 0 -> 2
- net -12V: track 42.7 -> 151.4 mm, vias 0 -> 1
- net B2: track 0.00 -> 108.4 mm, vias 0 -> 2
- net MAIN_OUT: track 5.61 -> 106.4 mm
- net B3: track 0.00 -> 100.2 mm, vias 0 -> 4
- net B6: track 0.00 -> 96.1 mm, vias 0 -> 1
- net B7: track 0.00 -> 85.2 mm, vias 0 -> 2
- net N$5: track 8.19 -> 93.3 mm
- net N$6: track 21.9 -> 101.8 mm
- net B5: track 8.79 -> 87.6 mm
- net CLOCKIN: track 74.7 -> 151.8 mm, vias 0 -> 3
- net B8: track 0.00 -> 59.9 mm
- net +12V: track 150.5 -> 207.7 mm, vias 1 -> 2
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- removed copper zone on layer 16, net GND
Other:
- board text added: "Music Thing Modular Turing Machine Rev 4 Prototype 1 March 2015 CC-BY-SA"
- board text removed: "&Reich"
- board text removed: "78L09->"
- board text removed: "Allen Strange"
- board text removed: "Cage"
- board text removed: "Designed in Herne Hill, London, May 2012 by Tom Whitwell"
- board text removed: "Dieter"
- board text removed: "Documentation: musicthing.co.uk/modular/"
- board text removed: "Doepfer"
- board text removed: "Don Buchla"
- board text removed: "Fredkin&Minsky"
- board text removed: "Glass"
- board text removed: "Grant Richter"
- board text removed: "Hal Chamberlin"
- board text removed: "Inspired"
- board text removed: "John"
- board text removed: "K.F.W"
- board text removed: "Ken Stone"
- board text removed: "Lunetta"
- board text removed: "Muffs"
- board text removed: "Navs"
- board text removed: "Nicholas Collins"
- board text removed: "Stanley"
- board text removed: "Turing Machine Random Looping Sequencer REV 4, March 2015"
- board text removed: "by:"
- board text removed: "|-R31 gain-|"

Commit message: Added BOM
Parts:
- R5: value 50k -> 51k
Changed lines of the file:
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@@
 <element name="R4" library="TomW" package="0207/7" value="100k" x="93.98" y="2.54"/>
 <element name="CV_IN" library="MusicThingModular" package="THONKICONN" value="THONKICONN" x="6.35" y="31.115" locked="yes" rot="R90"/>
-<element name="R5" library="TomW" package="0207/7" value="50k" x="5.715" y="24.765"/>
+<element name="R5" library="TomW" package="0207/7" value="51k" x="5.715" y="24.765"/>
 <element name="R6" library="TomW" package="0207/7" value="150k" x="69.85" y="12.7"/>
 <element name="CV_OUT" library="MusicThingModular" package="THONKICONN" value="THONKICONN" x="6.35" y="5.715" locked="yes" rot="R90"/>
