File: Hardware/TuringMachine.brd (EAGLE design)
At the start: 107 x 49.5 mm, 78 parts, among them IC1 TL072P, IC2 4015, IC3 4015, IC5 4016, IC6 TL072P, IC7 TL072P, T1 2N3904

Commit message: throwing smd parts on the board
Parts:
- removed EXPANSION: (no value), TomW:MA10-1
- removed POWER: (no value), TomW:MA05-2
- added 9, FUSE: FUSE, TomW:C050H075X075
- added D1, D3: 1N4001, SparkFun-DiscreteSemi:DIODE-HV
- added GATES, PULSES: (no value), con-lstb:MA08-2
- added IC10, IC9: 4050, 40xx:SO16
- added IC11, IC12: 78L09, linear:TO92
- added IC4, IC8: 4081, 40xx:SO14
- added POWER1: (no value), TomW:MA05-2
- C1, C12, C13, C14, C15, C16, C17, C2, C4, C7, C8, C9: device TomW:C050-024X044 -> SparkFun-Capacitors:0805
- C10, C11, C18: device rcl:C050-035X075 -> SparkFun-Capacitors:0805
- C5, C6: device SparkFun-Passives:CPOL-RADIAL-10UF-25V -> SparkFun-Capacitors:EIA3216
- D2: value 1N4148 -> BAT20JFILM; device MusicThingModular:DO35-7 -> SparkFun-DiscreteSemi:SOD-323
- IC1, IC6, IC7: value TL072P -> TL072_SMD; device TomW:DIL08 -> MusicThingModular:SO08
- IC2, IC3: device 40xx:DIL16 -> 40xx:SO16
- IC5: device 40xx:DIL14 -> 40xx:SO14
- R1, R10, R12, R13, R14, R15, R16, R18, R19, R2, R20, R22, R23, R24, R26, R27, R28, R29, R3, R30, R31, R32, R35, R5, R6, R7, R8, R9: device TomW:0207/7 -> SparkFun-Resistors:0805
- R11: device MusicThingModular:7MM_RESISTOR -> SparkFun-Resistors:0805
- T1: value 2N3904 -> (none); device transistor:TO92 -> transistor:SOT23-BEC
- U$2: value DAC0800 -> DAC0800SOIC; device TomW:DIL16 -> TomW:SO16
- moved R26 69.1 mm to (12.7, 2.54)
- moved C9 57.8 mm to (90.8, 3.81)
- moved D2 46.2 mm to (40.0, 20.3)
- moved R27 43.8 mm to (87.6, 5.08)
- moved IC7 42.3 mm to (45.7, 15.2), turned to 0 degrees
- moved R3 40.7 mm to (94.6, 3.81)
- moved R7 37.9 mm to (40.6, 25.4)
- moved C17 36.3 mm to (41.9, 22.9)
- moved R9 36.1 mm to (94.0, 7.62)
- moved C13 34.2 mm to (83.8, 3.81)
- moved C14 34.2 mm to (91.4, 7.62)
- moved C16 30.7 mm to (81.3, 6.35)
- moved R1 29.2 mm to (67.3, 6.35)
- moved R18 27.9 mm to (80.0, 3.81)
- moved R24 23.6 mm to (72.4, 6.35)
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Connections:
- new net CLOCK: GATES.10, GATES.9, IC10.6, IC4.9, IC8.13, IC8.2, IC8.6, IC8.8, PULSES.10, PULSES.9
- new net CLOCK2: IC10.10, IC4.13, IC4.2, IC4.6
- new net GATE1: GATES.1, IC10.15
- new net GATE2: GATES.2, IC10.12
- new net GATE3: GATES.3, IC10.2
- new net GATE4: GATES.4, IC10.4
- new net GATE5: GATES.5, IC9.12
- new net GATE6: GATES.6, IC9.10
- new net GATE7: GATES.7, IC9.6
- new net GATE8: GATES.8, IC9.2
- new net N$17: 9.2, POWER1.10, POWER1.9
- new net N$19: FUSE.2, POWER1.1, POWER1.2
- new net N$29: IC10.1, IC11.1
- new net N$38: IC12.1, IC9.1
- new net PULSE1: IC8.11, PULSES.1
- new net PULSE2: IC8.10, PULSES.2
- new net PULSE3: IC8.3, PULSES.3
- new net PULSE4: IC8.4, PULSES.4
- new net PULSE5: IC4.11, PULSES.5
- new net PULSE6: IC4.10, PULSES.6
- new net PULSE7: IC4.4, PULSES.7
- new net PULSE8: IC4.3, PULSES.8
- net +12V: now also 9.1, C5.A, D1.C, GATES.15, GATES.16, IC11.3, IC12.3, IC4.14, IC8.14, PULSES.15, PULSES.16; no longer C5.1, POWER.10, POWER.9
- net -12V: now also C6.C, D3.A, FUSE.1, GATES.11, GATES.12, PULSES.11, PULSES.12; no longer C6.2, POWER.1, POWER.2
- net B1: now also IC10.14, IC8.12; no longer EXPANSION.1
- net B2: now also IC10.11, IC8.9; no longer EXPANSION.2
- net B3: now also IC10.3, IC8.1; no longer EXPANSION.3
- net B4: now also IC10.5, IC8.5; no longer EXPANSION.4
- net B5: now also IC4.12, IC9.11; no longer EXPANSION.5
- net B6: now also IC4.8, IC9.9; no longer EXPANSION.6
- net B7: now also IC4.5, IC9.7; no longer EXPANSION.7
- net B8: now also IC4.1, IC9.3; no longer EXPANSION.8
- net CLOCKIN: now also D2.1, IC10.7, IC10.9; no longer D2.C, EXPANSION.10
- net GND: now also C5.C, C6.A, D1.A, D3.C, GATES.13, GATES.14, IC10.8, IC11.2, IC12.2, IC4.7, IC8.7, IC9.14, IC9.5, IC9.8, POWER1.3, POWER1.4, POWER1.5, POWER1.6, POWER1.7, POWER1.8, PULSES.13, PULSES.14, T1.B; no longer C5.2, C6.1, EXPANSION.9, POWER.3, POWER.4, POWER.5, POWER.6, POWER.7, POWER.8, T1.2
- net N$16: now also T1.E; no longer T1.3
- net N$8: now also D2.2; no longer D2.A
Routing:
- net GND: track 0.00 -> 512.6 mm, vias 0 -> 10
- net +12V: track 0.00 -> 337.6 mm, vias 0 -> 13
- net -12V: track 0.00 -> 269.9 mm, vias 0 -> 9
- net B1: track 0.00 -> 231.0 mm, vias 0 -> 8
- net CLOCKIN: track 0.00 -> 146.5 mm, vias 0 -> 9
- net CLOCK: track 0.00 -> 137.0 mm, vias 0 -> 9
- net B5: track 0.00 -> 136.8 mm, vias 0 -> 9
- net N$13: track 0.00 -> 136.6 mm
- net B6: track 0.00 -> 123.2 mm, vias 0 -> 7
- net B3: track 0.00 -> 119.3 mm, vias 0 -> 10
- net B4: track 0.00 -> 118.1 mm, vias 0 -> 12
- net N$6: track 0.00 -> 109.5 mm, vias 0 -> 3
- net START_OF_LOOP: track 0.00 -> 106.6 mm, vias 0 -> 10
- net B7: track 0.00 -> 104.7 mm, vias 0 -> 9
- net GATE1: track 0.00 -> 100.5 mm, vias 0 -> 1
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