File: Hardware/TuringBack.sch (EAGLE design)
At the start: 43 parts, among them IC11 78L09, IC12 78L09, IC7 TL072P

Commit message: Starting to route front board
Parts:
- BUS_1_BACK: device MusicThingModular:10PIN_BACKSIDE -> con-lstb:MA05-2
Changed lines of the file:
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@@
 <part name="C25" library="TomW" deviceset="C-EU" device="050-024X044" value="100n"/>
 <part name="BACK_BUS2" library="con-lstb" deviceset="MA03-2" device=""/>
-<part name="BUS_1_BACK" library="MusicThingModular" deviceset="10PIN_BACKSIDE" device=""/>
+<part name="BUS_1_BACK" library="con-lstb" deviceset="MA05-2" device=""/>
 </parts>
 <sheets>

Commit message: tidy up schematics
Other:
- note removed: "Channels between front and back: GND +12V -12V STEP_16_FRONT - STEP_16_BACK STEP_12_FRONT - STEP_12_BACK CLOCK_FRONT - CLOCK_BACK END_OF_LOOP_FRONT - END_OF_LOOP_BACKRL LOOP_CTRL_FRONT - LOOP_CTRL_BACK WRITE_SW_FRONT - START_OF_LOOP B1(-B8)_FRONT - B1(-B8)_BACK"
- note removed: "Power and expansion"
- note removed: "Randomised invert/loop switching"
