File: Hardware/TuringFront.sch (EAGLE design)
At the start: 71 parts, among them T1 2N3904, U1 TL074_

Commit message: Rev 4 Front and Back Boards complete
Parts:
- renumbered FRONT_BUS2 to LINK1, FRONT_PWR to LINK2, SV1 to LINK3
Changed lines of the file:
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@@
 <part name="C18" library="rcl" deviceset="C-EU" device="050-035X075" value="0.47uf"/>
 <part name="C12" library="TomW" deviceset="C-EU" device="050-024X044" value="1n"/>
-<part name="FRONT_PWR" library="MusicThingModular" deviceset="MA03-2BACKSIDE" device=""/>
+<part name="LINK2" library="MusicThingModular" deviceset="MA03-2BACKSIDE" device=""/>
 <part name="U1" library="MusicThingModular" deviceset="TL074" device="_"/>
-<part name="FRONT_BUS2" library="MusicThingModular" deviceset="MA03-2BACKSIDE" device=""/>
+<part name="LINK1" library="MusicThingModular" deviceset="MA03-2BACKSIDE" device=""/>
 <part name="PULSE_OUT" library="MusicThingModular" deviceset="THONKICONN" device="NEW"/>
 <part name="PULS1" library="TomW" deviceset="LED" device="3MM"/>
 <part name="R17" library="TomW" deviceset="R-EU_" device="0207/7" value="2.2k"/>
-<part name="SV1" library="MusicThingModular" deviceset="10PIN_BACKSIDE" device=""/>
+<part name="LINK3" library="MusicThingModular" deviceset="10PIN_BACKSIDE" device=""/>
 <part name="R1" library="TomW" deviceset="R-EU_" device="0207/7" value="2.2k"/>
 <part name="R4" library="TomW" deviceset="R-EU_" device="0207/7" value="2.2k"/>
@@
 <instance part="LENGTH" gate="G$1" x="68.58" y="25.4" rot="R90"/>
 <instance part="CHANGE" gate="G$1" x="66.04" y="228.6"/>
-<instance part="FRONT_PWR" gate="1" x="68.58" y="81.28"/>
-<instance part="FRONT_BUS2" gate="1" x="68.58" y="66.04"/>
-<instance part="SV1" gate="G$1" x="68.58" y="99.06"/>
+<instance part="LINK2" gate="1" x="68.58" y="81.28"/>
+<instance part="LINK1" gate="1" x="68.58" y="66.04"/>
+<instance part="LINK3" gate="G$1" x="68.58" y="99.06"/>
 <instance part="C7" gate="G$1" x="60.96" y="160.02"/>
 <instance part="C8" gate="G$1" x="60.96" y="142.24"/>
@@
 </segment>
 <segment>
-<pinref part="FRONT_PWR" gate="1" pin="6"/>
+<pinref part="LINK2" gate="1" pin="6"/>
 <wire x1="58.42" y1="83.82" x2="60.96" y2="83.82" width="0.1524" layer="91"/>
 <label x="58.42" y="83.82" size="1.016" layer="95" rot="R180" xref="yes"/>
 </segment>
 <segment>
-<pinref part="FRONT_PWR" gate="1" pin="5"/>
+<pinref part="LINK2" gate="1" pin="5"/>
 <wire x1="78.74" y1="83.82" x2="76.2" y2="83.82" width="0.1524" layer="91"/>
 <label x="78.74" y="83.82" size="1.016" layer="95" xref="yes"/>
@@
 </segment>
 <segment>
-<pinref part="FRONT_BUS2" gate="1" pin="2"/>
+<pinref part="LINK1" gate="1" pin="2"/>
 <wire x1="58.42" y1="63.5" x2="60.96" y2="63.5" width="0.1524" layer="91"/>
 <label x="58.42" y="63.5" size="1.016" layer="95" rot="R180" xref="yes"/>
@@
 </segment>
 <segment>
-<pinref part="FRONT_BUS2" gate="1" pin="3"/>
+<pinref part="LINK1" gate="1" pin="3"/>
 <wire x1="78.74" y1="66.04" x2="76.2" y2="66.04" width="0.1524" layer="91"/>
 <label x="78.74" y="66.04" size="1.016" layer="95" xref="yes"/>
@@
 </segment>
 <segment>
-<pinref part="FRONT_PWR" gate="1" pin="4"/>
+<pinref part="LINK2" gate="1" pin="4"/>
 <wire x1="58.42" y1="81.28" x2="60.96" y2="81.28" width="0.1524" layer="91"/>
 <label x="58.42" y="81.28" size="1.016" layer="95" rot="R180" xref="yes"/>
 </segment>
 <segment>
-<pinref part="FRONT_PWR" gate="1" pin="3"/>
+<pinref part="LINK2" gate="1" pin="3"/>
 <wire x1="78.74" y1="81.28" x2="76.2" y2="81.28" width="0.1524" layer="91"/>
 <label x="78.74" y="81.28" size="1.016" layer="95" xref="yes"/>
@@
 </segment>
 <segment>
-<pinref part="FRONT_PWR" gate="1" pin="2"/>
+<pinref part="LINK2" gate="1" pin="2"/>
 <wire x1="58.42" y1="78.74" x2="60.96" y2="78.74" width="0.1524" layer="91"/>
 <label x="58.42" y="78.74" size="1.016" layer="95" rot="R180" xref="yes"/>
 </segment>
 <segment>
-<pinref part="FRONT_PWR" gate="1" pin="1"/>
+<pinref part="LINK2" gate="1" pin="1"/>
 <wire x1="78.74" y1="78.74" x2="76.2" y2="78.74" width="0.1524" layer="91"/>
 <label x="78.74" y="78.74" size="1.016" layer="95" xref="yes"/>
@@
 </segment>
 <segment>
-<pinref part="FRONT_BUS2" gate="1" pin="5"/>
+<pinref part="LINK1" gate="1" pin="5"/>
 <wire x1="78.74" y1="68.58" x2="76.2" y2="68.58" width="0.1524" layer="91"/>
 <label x="78.74" y="68.58" size="1.016" layer="95" xref="yes"/>
@@
 </segment>
 <segment>
-<pinref part="FRONT_BUS2" gate="1" pin="6"/>
+<pinref part="LINK1" gate="1" pin="6"/>
 <wire x1="58.42" y1="68.58" x2="60.96" y2="68.58" width="0.1524" layer="91"/>
 <label x="58.42" y="68.58" size="1.016" layer="95" rot="R180" xref="yes"/>
@@
 <wire x1="78.74" y1="93.98" x2="76.2" y2="93.98" width="0.1524" layer="91"/>
 <label x="78.74" y="93.98" size="1.016" layer="95" xref="yes"/>
-<pinref part="SV1" gate="G$1" pin="1"/>
+<pinref part="LINK3" gate="G$1" pin="1"/>
 </segment>
 <segment>
@@
 <wire x1="78.74" y1="96.52" x2="76.2" y2="96.52" width="0.1524" layer="91"/>
 <label x="78.74" y="96.52" size="1.016" layer="95" xref="yes"/>
-<pinref part="SV1" gate="G$1" pin="3"/>
+<pinref part="LINK3" gate="G$1" pin="3"/>
 </segment>
 <segment>
@@
 <wire x1="58.42" y1="96.52" x2="60.96" y2="96.52" width="0.1524" layer="91"/>
 <label x="58.42" y="96.52" size="1.016" layer="95" rot="R180" xref="yes"/>
-<pinref part="SV1" gate="G$1" pin="4"/>
+<pinref part="LINK3" gate="G$1" pin="4"/>
 </segment>
 <segment>
@@
 <wire x1="78.74" y1="99.06" x2="76.2" y2="99.06" width="0.1524" layer="91"/>
 <label x="78.74" y="99.06" size="1.016" layer="95" xref="yes"/>
-<pinref part="SV1" gate="G$1" pin="5"/>
+<pinref part="LINK3" gate="G$1" pin="5"/>
 </segment>
 <segment>
@@
 <wire x1="58.42" y1="99.06" x2="60.96" y2="99.06" width="0.1524" layer="91"/>
 <label x="58.42" y="99.06" size="1.016" layer="95" rot="R180" xref="yes"/>
-<pinref part="SV1" gate="G$1" pin="6"/>
+<pinref part="LINK3" gate="G$1" pin="6"/>
 </segment>
 <segment>
@@
 <wire x1="78.74" y1="101.6" x2="76.2" y2="101.6" width="0.1524" layer="91"/>
 <label x="78.74" y="101.6" size="1.016" layer="95" xref="yes"/>
-<pinref part="SV1" gate="G$1" pin="7"/>
+<pinref part="LINK3" gate="G$1" pin="7"/>
 </segment>
 <segment>
@@
 </segment>
 <segment>
-<pinref part="FRONT_BUS2" gate="1" pin="4"/>
+<pinref part="LINK1" gate="1" pin="4"/>
 <wire x1="58.42" y1="66.04" x2="60.96" y2="66.04" width="0.1524" layer="91"/>
 <label x="58.42" y="66.04" size="1.016" layer="95" rot="R180" xref="yes"/>
@@
 <wire x1="58.42" y1="93.98" x2="60.96" y2="93.98" width="0.1524" layer="91"/>
 <label x="58.42" y="93.98" size="1.016" layer="95" rot="R180" xref="yes"/>
-<pinref part="SV1" gate="G$1" pin="2"/>
+<pinref part="LINK3" gate="G$1" pin="2"/>
 </segment>
 <segment>
@@
 <wire x1="58.42" y1="101.6" x2="60.96" y2="101.6" width="0.1524" layer="91"/>
 <label x="58.42" y="101.6" size="1.016" layer="95" rot="R180" xref="yes"/>
-<pinref part="SV1" gate="G$1" pin="8"/>
+<pinref part="LINK3" gate="G$1" pin="8"/>
 </segment>
 <segment>
@@
 <wire x1="78.74" y1="104.14" x2="76.2" y2="104.14" width="0.1524" layer="91"/>
 <label x="78.74" y="104.14" size="1.016" layer="95" xref="yes"/>
-<pinref part="SV1" gate="G$1" pin="9"/>
+<pinref part="LINK3" gate="G$1" pin="9"/>
 </segment>
 <segment>
@@
 <net name="NOISE_FRONT" class="0">
 <segment>
-<pinref part="FRONT_BUS2" gate="1" pin="1"/>
+<pinref part="LINK1" gate="1" pin="1"/>
 <wire x1="78.74" y1="63.5" x2="76.2" y2="63.5" width="0.1524" layer="91"/>
 <label x="78.74" y="63.5" size="1.016" layer="95" xref="yes"/>
@@
 <wire x1="58.42" y1="104.14" x2="60.96" y2="104.14" width="0.1524" layer="91"/>
 <label x="58.42" y="104.14" size="1.016" layer="95" rot="R180" xref="yes"/>
-<pinref part="SV1" gate="G$1" pin="10"/>
-</segment>
-<segment>
+<pinref part="LINK3" gate="G$1" pin="10"/>
+</segment>
+<segment>

Commit message: Finalised V4 PCBs
Other:
- moved on the sheet: C14, C16, C7, C8, C9
Changed lines of the file:
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@@
 <part name="WRITE" library="TomW" deviceset="T-80-T-SPDT-ON-OFF-ON" device=""/>
 <part name="R18" library="TomW" deviceset="R-EU_" device="0207/7" value="1k"/>
-<part name="GND18" library="supply1" deviceset="GND" device=""/>
 <part name="R22" library="TomW" deviceset="R-EU_" device="0207/7" value="100k"/>
 <part name="R23" library="TomW" deviceset="R-EU_" device="0207/7" value="10k"/>
@@
 <instance part="LINK1" gate="1" x="68.58" y="66.04"/>
 <instance part="LINK3" gate="G$1" x="68.58" y="99.06"/>
-<instance part="C7" gate="G$1" x="60.96" y="160.02"/>
-<instance part="C8" gate="G$1" x="60.96" y="142.24"/>
+<instance part="C7" gate="G$1" x="60.96" y="160.02" rot="R180"/>
+<instance part="C8" gate="G$1" x="60.96" y="142.24" rot="R180"/>
 <instance part="C13" gate="G$1" x="71.12" y="160.02"/>
 <instance part="T1" gate="G1" x="144.78" y="81.28" rot="R180"/>
@@
 <instance part="R7" gate="G$1" x="340.36" y="93.98" rot="R180"/>
 <instance part="C15" gate="G$1" x="309.88" y="76.2" rot="R180"/>
-<instance part="C16" gate="G$1" x="345.44" y="68.58"/>
-<instance part="C14" gate="G$1" x="71.12" y="139.7" rot="R180"/>
+<instance part="C16" gate="G$1" x="345.44" y="68.58" rot="R180"/>
+<instance part="C14" gate="G$1" x="71.12" y="139.7"/>
 <instance part="U$2" gate="G$1" x="210.82" y="193.04" rot="R180"/>
 <instance part="R26" gate="G$1" x="243.84" y="157.48"/>
 <instance part="R27" gate="G$1" x="243.84" y="208.28" rot="R180"/>
 <instance part="R28" gate="G$1" x="243.84" y="226.06"/>
-<instance part="C9" gate="G$1" x="246.38" y="195.58" rot="R270"/>
+<instance part="C9" gate="G$1" x="246.38" y="195.58" rot="R90"/>
 <instance part="U1" gate="A" x="246.38" y="167.64"/>
-<instance part="GND18" gate="1" x="233.68" y="167.64"/>
 <instance part="CV_OUT" gate="G$1" x="292.1" y="157.48"/>
 <instance part="U1" gate="D" x="218.44" y="93.98"/>
@@
 <wire x1="71.12" y1="170.18" x2="81.28" y2="170.18" width="0.1524" layer="91"/>
 <pinref part="C7" gate="G$1" pin="2"/>
-<wire x1="60.96" y1="154.94" x2="60.96" y2="170.18" width="0.1524" layer="91"/>
+<wire x1="60.96" y1="165.1" x2="60.96" y2="170.18" width="0.1524" layer="91"/>
 <junction x="60.96" y="170.18"/>
 <pinref part="C13" gate="G$1" pin="1"/>
@@
 </segment>
 </net>
-<net name="END_OF_LOOP_BACK" class="0">
-<segment>
-<wire x1="48.26" y1="22.86" x2="43.18" y2="22.86" width="0.1524" layer="91"/>
-<label x="43.18" y="22.86" size="1.016" layer="95" rot="R180" xref="yes"/>
-</segment>
-</net>
 <net name="N$3" class="0">
 <segment>
@@
 <wire x1="60.96" y1="149.86" x2="71.12" y2="149.86" width="0.1524" layer="91"/>
 <pinref part="C7" gate="G$1" pin="1"/>
-<wire x1="60.96" y1="162.56" x2="60.96" y2="149.86" width="0.1524" layer="91"/>
+<wire x1="60.96" y1="157.48" x2="60.96" y2="149.86" width="0.1524" layer="91"/>
 <junction x="60.96" y="149.86"/>
 <pinref part="C13" gate="G$1" pin="2"/>
@@
 <junction x="71.12" y="149.86"/>
 <pinref part="C8" gate="G$1" pin="2"/>
-<wire x1="60.96" y1="137.16" x2="60.96" y2="149.86" width="0.1524" layer="91"/>
+<wire x1="60.96" y1="147.32" x2="60.96" y2="149.86" width="0.1524" layer="91"/>
 <pinref part="C14" gate="G$1" pin="1"/>
-<wire x1="71.12" y1="137.16" x2="71.12" y2="149.86" width="0.1524" layer="91"/>
+<wire x1="71.12" y1="142.24" x2="71.12" y2="149.86" width="0.1524" layer="91"/>
 <wire x1="49.53" y1="149.86" x2="60.96" y2="149.86" width="0.1524" layer="91"/>
 <label x="49.53" y="149.86" size="1.016" layer="95" rot="R180" xref="yes"/>
@@
 <junction x="330.2" y="60.96"/>
 <pinref part="C16" gate="G$1" pin="1"/>
-<wire x1="345.44" y1="60.96" x2="345.44" y2="71.12" width="0.1524" layer="91"/>
+<wire x1="345.44" y1="60.96" x2="345.44" y2="66.04" width="0.1524" layer="91"/>
 <label x="330.2" y="59.69" size="1.016" layer="95" rot="R270" xref="yes"/>
 </segment>
@@
 </segment>
 <segment>
-<pinref part="U1" gate="A" pin="+IN"/>
-<pinref part="GND18" gate="1" pin="GND"/>
-<wire x1="238.76" y1="170.18" x2="233.68" y2="170.18" width="0.1524" layer="91"/>
-</segment>
-<segment>
 <wire x1="254" y1="205.74" x2="254" y2="208.28" width="0.1524" layer="91"/>
 <pinref part="R27" gate="G$1" pin="1"/>
@@
 <junction x="124.46" y="144.78"/>
 </segment>
+<segment>
+<pinref part="U1" gate="A" pin="+IN"/>
+<wire x1="236.22" y1="170.18" x2="238.76" y2="170.18" width="0.1524" layer="91"/>
+<label x="236.22" y="170.18" size="1.778" layer="95" rot="R90" xref="yes"/>
+</segment>
 </net>
 <net name="-12V_FRONT" class="1">
@@
 <wire x1="71.12" y1="129.54" x2="81.28" y2="129.54" width="0.1524" layer="91"/>
 <pinref part="C8" gate="G$1" pin="1"/>
-<wire x1="60.96" y1="144.78" x2="60.96" y2="129.54" width="0.1524" layer="91"/>
+<wire x1="60.96" y1="139.7" x2="60.96" y2="129.54" width="0.1524" layer="91"/>
 <junction x="60.96" y="129.54"/>
 <pinref part="C14" gate="G$1" pin="2"/>
-<wire x1="71.12" y1="144.78" x2="71.12" y2="129.54" width="0.1524" layer="91"/>
+<wire x1="71.12" y1="134.62" x2="71.12" y2="129.54" width="0.1524" layer="91"/>
 <junction x="71.12" y="129.54"/>
 <label x="48.26" y="129.54" size="1.016" layer="95" rot="R180" xref="yes"/>
@@
 <wire x1="254" y1="190.5" x2="223.52" y2="190.5" width="0.1524" layer="91"/>
 <pinref part="C9" gate="G$1" pin="2"/>
-<wire x1="241.3" y1="195.58" x2="254" y2="195.58" width="0.1524" layer="91"/>
+<wire x1="251.46" y1="195.58" x2="254" y2="195.58" width="0.1524" layer="91"/>
 <wire x1="254" y1="195.58" x2="254" y2="190.5" width="0.1524" layer="91"/>
 <label x="255.27" y="185.42" size="1.016" layer="95" xref="yes"/>
@@
 <junction x="330.2" y="76.2"/>
 <pinref part="C16" gate="G$1" pin="2"/>
-<wire x1="345.44" y1="76.2" x2="345.44" y2="63.5" width="0.1524" layer="91"/>
+<wire x1="345.44" y1="76.2" x2="345.44" y2="73.66" width="0.1524" layer="91"/>
 </segment>
 </net>
@@
 <pinref part="U$2" gate="G$1" pin="COMP"/>
 <pinref part="C9" gate="G$1" pin="1"/>
-<wire x1="223.52" y1="195.58" x2="248.92" y2="195.58" width="0.1524" layer="91"/>
-</segment>
-</net>
+<wire x1="223.52" y1="195.58" x2="243.84" y2="195.58" width="0.1524" layer="91"/>
+</segment>
+</net>

Commit message: Front board updated with new Write switch component
Slightly enlarged holes to accommodate 2.03 x 0.76 solder tags
Parts:
- WRITE: device TomW:T-80-T-SPDT-ON-OFF-ON -> MusicThingModular:T-80-T-SPDT-ON-OFF-ON
Changed lines of the file:
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@@
 <part name="R3" library="TomW" deviceset="R-EU_" device="0207/7" value="68k"/>
 <part name="R9" library="TomW" deviceset="R-EU_" device="0207/7" value="15k"/>
-<part name="WRITE" library="TomW" deviceset="T-80-T-SPDT-ON-OFF-ON" device=""/>
+<part name="WRITE" library="MusicThingModular" deviceset="T-80-T-SPDT-ON-OFF-ON" device=""/>
 <part name="R18" library="TomW" deviceset="R-EU_" device="0207/7" value="1k"/>
 <part name="R22" library="TomW" deviceset="R-EU_" device="0207/7" value="100k"/>
